File: hardware/KiCad/SwasthEdge/SwasthEdge.kicad_pcb (KiCad board)
At the start: 2 copper layers, 100 x 100 mm, 89 parts, among them J1 Conn_01x02, J2 Conn_01x04, J3 Conn_01x03, J4 Micro_SD_Card_Det1, J5 Conn_01x05, J6 Conn_02x04_Counter_Clockwise, J7 LOAD_OUT, K1 SRD-05VDC-SL-C, U1 LM2596S-5, U10 ULN2003ADR, U12 STM32F446RETx, U2 AMS1117-3.3, U3 DS3231SN, U4 INA226, U5 SHT31-DIS, U6 W25Q64JVSSIQ, U7 MCP4131-103E/SN, U8 MAX13487EESA, U9 TPS3813K33DBVR, Y1 8MHz

Commit message: Update SwasthEdge KiCad board with routed PCB
Parts:
- BT1: footprint Battery:BatteryHolder_Keystone_3000_1xCR2032 -> BatteryHolder_Keystone_3000_1xCR2032
- H1, H2, H3, H4: footprint MountingHole:MountingHole_3.2mm_M3_Pad -> MountingHole_3.2mm_M3_Pad
- moved R14 63.8 mm to (111.0, 102.5)
- moved D7 49.6 mm to (111.0, 107.0)
- moved TP3 49.0 mm to (160.0, 128.0)
- moved C9 45.3 mm to (131.0, 144.0)
- moved R10 39.7 mm to (137.0, 110.5)
- moved R6 37.4 mm to (131.5, 110.0), turned to 0 degrees
- moved C10 36.9 mm to (110.0, 118.0)
- moved D10 36.4 mm to (137.0, 115.0)
- moved TP2 33.5 mm to (155.0, 128.0)
- moved TP1 30.7 mm to (150.0, 56.5)
- moved D6 30.3 mm to (163.0, 110.0)
- moved R17 27.3 mm to (162.0, 137.0)
- moved R12 21.4 mm to (160.0, 123.5), turned to 0 degrees
- moved C8 18.8 mm to (132.5, 125.0)
- moved TP6 14.5 mm to (132.5, 129.5)
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Routing:
- net GND: track 0.00 -> 804.8 mm, vias 0 -> 82
- net +3V3: track 0.00 -> 456.9 mm, vias 0 -> 66
- net +5V: track 0.00 -> 262.3 mm, vias 0 -> 19
- net /POWER_RAIL: track 0.00 -> 144.0 mm, vias 0 -> 9
- net /SENSOR_VCC: track 0.00 -> 108.7 mm, vias 0 -> 3
- net /I2C1_SDA: track 0.00 -> 106.4 mm, vias 0 -> 9
- net /I2C1_SCL: track 0.00 -> 93.2 mm, vias 0 -> 7
- net +12V: track 0.00 -> 87.2 mm, vias 0 -> 8
- net /NRST: track 0.00 -> 85.3 mm, vias 0 -> 7
- net /SPI1_MOSI: track 0.00 -> 85.2 mm, vias 0 -> 9
- net /FAULT_DISC: track 0.00 -> 77.6 mm, vias 0 -> 3
- net /SPI1_SCK: track 0.00 -> 77.5 mm, vias 0 -> 7
- net /CS_SD: track 0.00 -> 72.0 mm, vias 0 -> 6
- net /FAULT_COMM: track 0.00 -> 71.5 mm, vias 0 -> 3
- net /FAULT_CURR: track 0.00 -> 65.6 mm, vias 0 -> 2
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Other:
- copper layers 2 -> 4
